Commit message: Correcciones Parte 1, no completado

File: ros2_ws_mecanum_estudiantes/ros2_ws_mecanum/install/mi_robot_mecanum/share/mi_robot_mecanum/urdf/mi_robot.urdf.xacro (robot description, xacro)
@@ -64,4 +64,10 @@
       <!-- TODO: <inertial> de un cilindro de masa rueda_masa, radio rueda_radio y largo rueda_ancho -->
     </link>
+    <joint name="joint_rueda_${prefijo}" type="continuous">
+      <parent link="base_link"/>
+      <child link="rueda_${prefijo}"/>
+      <origin xyz="${x_signo * separacion_ruedas/2} ${y_signo * separacion_ruedas/2} -0.02" rpy="-1.5708 0 0"/>
+      <axis xyz="0 0 1"/>
+    </joint>
     <!-- TODO: joint "joint_rueda_${prefijo}" tipo continuous entre base_link y
          rueda_${prefijo}, en (x_signo*lx, y_signo*ly, 0). Igual que en el diferencial:
@@ -76,10 +82,29 @@
   <!-- TODO: link "lidar_link" (cilindro) con dimensiones y masa de la hoja de datos:
        visual, collision e inertial -->
+  <link name="lidar_link">
+      <origin xyz="0 0 0.14" rpy="0 0 0"/>
+      <visual>
+        <geometry><cylinder radius="0.038" length="0.041"/></geometry>
+        <material name="negro"><color rgba="0.1 0.1 0.1 1"/></material>
+      </visual>
+      <origin xyz="0 0 0.14" rpy="0 0 0"/>
+      <collision>
+        <geometry><sphere radius="0.038"/></geometry>
+      </collision>
+      <inertial>
+        <xacro:inercia_cilindro m="0.190" r="0.038" h="0.041"/>
+      </inertial>
+  </link>
+  <joint name="joint_lidar" type="fixed">
+    <parent link="base_link"/>
+    <child link="lidar_link"/>
+    <origin xyz="0 0 0.14" rpy="0 0 0"/>
+  </joint>
   <!-- TODO: joint fijo "joint_lidar" base_link -> lidar_link en la posición de su variante -->
   <gazebo reference="lidar_link">
     <sensor name="rplidar_a3" type="gpu_lidar">
       <topic>/scan</topic>
-      <gz_frame_id>TODO</gz_frame_id>
-      <update_rate>TODO</update_rate>
+      <gz_frame_id>lidar_link</gz_frame_id>
+      <update_rate>10</update_rate>
       <always_on>1</always_on>
       <visualize>true</visualize>
@@ -87,13 +112,13 @@
         <scan>
           <horizontal>
-            <samples>TODO</samples>          <!-- muestras por vuelta -->
+            <samples>360</samples>          <!-- muestras por vuelta -->
             <resolution>1</resolution>
-            <min_angle>TODO</min_angle>
-            <max_angle>TODO</max_angle>
+            <min_angle>-3.14159</min_angle>
+            <max_angle>3.14159</max_angle>
           </horizontal>
         </scan>
         <range>
-          <min>TODO</min>
-          <max>TODO</max>
+          <min>0.2</min>
+          <max>4</max>
           <resolution>0.01</resolution>
         </range>
@@ -104,5 +129,31 @@
   <!-- ===================== Orbbec Astra (Parte 2) ===================== -->
   <!-- TODO: link "camara_link" (caja) con dimensiones y masa de la hoja de datos -->
+  <link name="camara_link">
+    <visual>
+      <origin xyz="0.14 0 0.08" rpy="0 0 0"/>
+      <geometry><box size="0.040 0.165 0.048"/></geometry>
+      <material name="red"><color rgba="1 0.1 0.1 1"/></material>
+    </visual>
+    <collision>
+      <origin xyz="0.14 0 0.08" rpy="0 0 0"/>
+      <geometry><box size="0.040 0.165 0.048"/></geometry>
+    </collision>
+    <inertial>
+      <origin xyz="0.14 0 0.08" rpy="0 0 0"/>
+      <mass value="0.310"/>
+      <xacro:inercia_caja m="0.310" x="0.040" y="0.165" z="0.048"/>
+    </inertial>
+  </link>
+  <joint name="joint_camara" type="fixed">
+    <parent link="base_link"/>
+    <child link="camara_link"/>
+    <origin xyz="0.14 0 0.08" rpy="0 0 0"/>
+  </joint>
   <!-- TODO: joint fijo "joint_camara" base_link -> camara_link en la posición de su variante -->
+  <joint name="joint_camara_optica" type="fixed">
+    <parent link="base_link"/>
+    <child link="camara_optica_link"/>
+    <origin xyz="0.14 0 0.08" rpy="-pi/2 0 pi/2"/>
+  </joint>
   <!-- TODO: link "camara_optica_link" y joint fijo "joint_camara_optica" desde
        camara_link con rpy = (-π/2, 0, -π/2) (REP-103) -->
@@ -110,22 +161,22 @@
     <sensor name="astra" type="rgbd_camera">
       <topic>/camara</topic>
-      <gz_frame_id>TODO</gz_frame_id>
-      <update_rate>TODO</update_rate>
+      <gz_frame_id>camara_link</gz_frame_id>
+      <update_rate>10</update_rate>
       <always_on>1</always_on>
       <camera>
-        <horizontal_fov>TODO</horizontal_fov>   <!-- en radianes -->
+        <horizontal_fov>1.047</horizontal_fov>   <!-- en radianes -->
         <image>
-          <width>TODO</width>
-          <height>TODO</height>
+          <width>640</width>
+          <height>480</height>
           <format>R8G8B8</format>
         </image>
         <clip>
-          <near>TODO</near>
-          <far>TODO</far>
+          <near>0.6</near>
+          <far>8</far>
         </clip>
         <depth_camera>
           <clip>
-            <near>TODO</near>
-            <far>TODO</far>
+            <near>0.6</near>
+            <far>8</far>
           </clip>
         </depth_camera>
@@ -145,5 +196,11 @@
   <gazebo>
     <xacro:motor prefijo="del_izq"/>
+    <xacro:motor prefijo="tra_izq"/>
+    <xacro:motor prefijo="del_der"/>
+    <xacro:motor prefijo="tra_der"/>
     <!-- TODO: motores de del_der, tra_izq y tra_der -->
+    <plugin filename="gz-sim-joint-state-publisher-system" name="gz::sim::systems::JointStatePublisher"> <!-- JointState plugin only to publish data from gazebo-->
+      <topic>joint_states</topic>
+    </plugin>
     <!-- TODO: plugin gz-sim-joint-state-publisher-system (encoders) -->
   </gazebo>

File: ros2_ws_mecanum_estudiantes/ros2_ws_mecanum/src/mi_robot_mecanum/urdf/mi_robot.urdf.xacro (robot description, xacro)
@@ -212,5 +212,11 @@
   <gazebo>
     <xacro:motor prefijo="del_izq"/>
+    <xacro:motor prefijo="tra_izq"/>
+    <xacro:motor prefijo="del_der"/>
+    <xacro:motor prefijo="tra_der"/>
     <!-- TODO: motores de del_der, tra_izq y tra_der -->
+    <plugin filename="gz-sim-joint-state-publisher-system" name="gz::sim::systems::JointStatePublisher"> <!-- JointState plugin only to publish data from gazebo-->
+      <topic>joint_states</topic>
+    </plugin>
     <!-- TODO: plugin gz-sim-joint-state-publisher-system (encoders) -->
   </gazebo>
